File: Loom23/CLT.kicad_sch (KiCad schematic)
At the start: 0 parts

Commit message: Added detailed version of schematic
Parts:
- added TH?: (no value), symbol Device:Thermistor_NTC
Connections:
- new net CLTSIG: TH?.2
- new net SENGND: TH?.1
Changed lines of the file:
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@@
 (kicad_sch (version 20211123) (generator eeschema)
   (paper "A4")
+  (wire (pts (xy 133.35 93.98) (xy 137.16 93.98))
+    (stroke (width 0) (type default) (color 0 0 0 0))
+  )
+  (wire (pts (xy 144.78 93.98) (xy 148.59 93.98))
+    (stroke (width 0) (type default) (color 0 0 0 0))
+  )
+  (hierarchical_label "SENGND" (shape input) (at 133.35 93.98 180)
+    (effects (font (size 1.27 1.27)) (justify right))
+  )
+  (hierarchical_label "CLTSIG" (shape input) (at 148.59 93.98 0)
+    (effects (font (size 1.27 1.27)) (justify left))
+  )
+  (symbol (lib_id "Device:Thermistor_NTC") (at 140.97 93.98 90) (unit 1)
+    (in_bom yes) (on_board yes) (fields_autoplaced)
+    (property "Reference" "TH?" (id 0) (at 141.2875 87.63 90))
+    (property "Value" "" (id 1) (at 141.2875 90.17 90))
+    (property "Footprint" "" (id 2) (at 139.7 93.98 0)
+      (effects (font (size 1.27 1.27)) hide)
+    )
+    (property "Datasheet" "~" (id 3) (at 139.7 93.98 0)
+      (effects (font (size 1.27 1.27)) hide)
+    )
+    (pin "1")
+    (pin "2")
+  )
 )

Commit message: Signed-off-by: fst29 <fst29@cam.ac.uk>
Parts:
- TH?: value (none) -> Thermistor_NTC
Changed lines of the file:
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@@
     (in_bom yes) (on_board yes) (fields_autoplaced)
     (property "Reference" "TH?" (id 0) (at 141.2875 87.63 90))
-    (property "Value" "" (id 1) (at 141.2875 90.17 90))
+    (property "Value" "Thermistor_NTC" (id 1) (at 141.2875 90.17 90))
     (property "Footprint" "" (id 2) (at 139.7 93.98 0)
       (effects (font (size 1.27 1.27)) hide)
