File: Loom23/Starter relay and switch.kicad_sch (KiCad schematic)
At the start: 0 parts

Commit message: Included BSPD and started adding labels
Parts:
- added K?: DIPxx-1Axx-11x, Relay_THT:Relay_StandexMeder_DIP_LowProfile, symbol Relay:DIPxx-1Axx-11x
Connections:
- new net +12V: K?.7, K?.8
- new net GND: K?.2
- new net Starter Signal: K?.6
- new net StarterPower: K?.1, K?.14
Changed lines of the file:
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@@
 (kicad_sch (version 20211123) (generator eeschema)
   (paper "A4")
+  (wire (pts (xy 158.75 73.66) (xy 165.1 73.66))
+    (stroke (width 0) (type default) (color 0 0 0 0))
+  )
+  (wire (pts (xy 158.75 83.82) (xy 165.1 83.82))
+    (stroke (width 0) (type default) (color 0 0 0 0))
+  )
+  (wire (pts (xy 134.62 73.66) (xy 143.51 73.66))
+    (stroke (width 0) (type default) (color 0 0 0 0))
+  )
+  (wire (pts (xy 139.7 83.82) (xy 143.51 83.82))
+    (stroke (width 0) (type default) (color 0 0 0 0))
+  )
+  (hierarchical_label "Starter Signal" (shape input) (at 139.7 83.82 180)
+    (effects (font (size 1.27 1.27)) (justify right))
+  )
+  (hierarchical_label "StarterPower" (shape input) (at 165.1 73.66 0)
+    (effects (font (size 1.27 1.27)) (justify left))
+  )
+  (hierarchical_label "GND" (shape input) (at 165.1 83.82 0)
+    (effects (font (size 1.27 1.27)) (justify left))
+  )
+  (hierarchical_label "+12V" (shape input) (at 134.62 73.66 180)
+    (effects (font (size 1.27 1.27)) (justify right))
+  )
+  (symbol (lib_id "Relay:DIPxx-1Axx-11x") (at 151.13 78.74 90) (unit 1)
+    (in_bom yes) (on_board yes) (fields_autoplaced)
+    (property "Reference" "K?" (id 0) (at 151.13 66.04 90))
+    (property "Value" "DIPxx-1Axx-11x" (id 1) (at 151.13 68.58 90))
+    (property "Footprint" "Relay_THT:Relay_StandexMeder_DIP_LowProfile" (id 2) (at 152.4 69.85 0)
+      (effects (font (size 1.27 1.27)) (justify left) hide)
+    )
+    (property "Datasheet" "https://standexelectronics.com/wp-content/uploads/datasheet_reed_relay_DIP.pdf" (id 3) (at 151.13 78.74 0)
+      (effects (font (size 1.27 1.27)) hide)
+    )
+    (pin "1")
+    (pin "14")
+    (pin "2")
+    (pin "6")
+    (pin "7")
+    (pin "8")
+  )
 )
