File: Loom23/BSPD.kicad_sch (KiCad schematic)
At the start: 0 parts

Commit message: Included BSPD and started adding labels
Parts:
- added C1, C7: 1uF, Capacitor_THT:CP_Radial_D5.0mm_P2.00mm, symbol Device:C_Polarized
- added C10, C11: 10uF, Capacitor_THT:C_Disc_D6.0mm_W4.4mm_P5.00mm, symbol Device:C
- added C2, C8: 0.01uF, Capacitor_THT:C_Disc_D6.0mm_W2.5mm_P5.00mm, symbol Device:C
- added C3: 0.33uF, Capacitor_THT:CP_Radial_D5.0mm_P2.00mm, symbol Device:C_Polarized
- added C4: 0.1uF, Capacitor_THT:CP_Radial_D5.0mm_P2.00mm, symbol Device:C_Polarized
- added C5, C6, C9: 0.1uF, Capacitor_THT:C_Disc_D6.0mm_W2.5mm_P5.00mm, symbol Device:C
- added D1, D3, D4: 1N5817, Diode_THT:D_DO-41_SOD81_P10.16mm_Horizontal, symbol Diode:1N4001
- added D2, D5, D6, D7: LED, LED_THT:LED_D5.0mm, symbol Device:LED
- added J1, J2, J3: Test Pad, Additional Footprints:TestPad, symbol Connector:Conn_01x01_Female
- added J4, J6: 282087-1, Additional Footprints:3 pin flying lead, symbol Connector:Conn_01x03_Female
- added J5: 282105-1, Additional Footprints:3 pin flying lead, symbol Connector:Conn_01x03_Female
- added K1: MCCMA51-S-DC12V-C, Additional Footprints:MCCMA51-S-DC12V-C, symbol Additional_Components:Relay
- added Q1: IRLZ44Z, Additional Footprints:TO-220-TabDown-NoHole, symbol Transistor_FET:IRLZ44N
- added R1, R13, R15, R16, R18, R2, R3, R4, R5, R6: 1k, Resistor_THT:R_Axial_DIN0207_L6.3mm_D2.5mm_P7.62mm_Horizontal, symbol Device:R
- added R10: 4.7k, Resistor_THT:R_Axial_DIN0207_L6.3mm_D2.5mm_P7.62mm_Horizontal, symbol Device:R
- added R11, R14, R17, R20, R21, R8: 220R, Resistor_THT:R_Axial_DIN0207_L6.3mm_D2.5mm_P7.62mm_Horizontal, symbol Device:R
- added R12: 1.6Meg, Resistor_THT:R_Axial_DIN0207_L6.3mm_D2.5mm_P7.62mm_Horizontal, symbol Device:R
- added R19, R7: 5Meg, Resistor_THT:R_Axial_DIN0207_L6.3mm_D2.5mm_P7.62mm_Horizontal, symbol Device:R
- added R9: 56k, Resistor_THT:R_Axial_DIN0207_L6.3mm_D2.5mm_P7.62mm_Horizontal, symbol Device:R
- added RV1, RV2, RV3, RV4: 10k, Potentiometer_THT:Potentiometer_Bourns_3296Y_Vertical, symbol Device:R_Potentiometer
- added U1: LM7805_TO220, Additional Footprints:TO-220-TabDown-NoHole, symbol Regulator_Linear:LM7805_TO220
- added U2: 4011, Package_DIP:DIP-14_W7.62mm_LongPads, symbol 4xxx:4011
- added U3: 4081, Package_DIP:DIP-14_W7.62mm_LongPads, symbol 4xxx:4081
- added U4, U5, U6: MCP6542, Package_DIP:DIP-8_W7.62mm_LongPads, symbol Additional_Components:MCP6542
Connections:
- new net: R3.1, U3.12
- new net: D7.2 (A), R21.1
- new net: R21.2, U3.2, U6.7
- new net: J1.1 (Pin_1), U3.10
- new net: R1.1, U3.8
- new net: R2.1, U3.9
- new net: J5.2 (Pin_2), K1.3
- new net: R13.2, R15.1, U4.2 (-)
- new net: D3.2 (A), R9.1, U2.3
- new net: C10.1, R11.2, R9.2, U4.3 (+)
- new net: D1.2 (A), K1.1, Q1.2 (D)
- new net: D3.1 (K), R11.1
- new net: J3.1 (Pin_1), U2.10
- new net: D6.2 (A), R20.1
- new net: R20.2, U3.1, U6.1
- new net: D4.1 (K), R12.1, U2.12, U4.1
- new net: R5.1, U2.8
- new net: R6.1, U2.9
- new net: D2.2 (A), R8.1
- new net: D4.2 (A), R14.1
- new net: C11.1, R12.2, R14.2, U4.5 (+)
- new net: RV4.2, U6.5 (+)
- new net: Q1.1 (G), R10.2
- new net: R16.2, R18.1, U4.6 (-)
- new net: U2.13, U4.7
- new net: J2.1 (Pin_1), U3.11
- new net: R4.1, U3.13
- new net: RV2.2, U5.5 (+)
- new net: R8.2, U2.1, U5.1
- new net: R17.2, U2.2, U5.7
- new net: RV3.2, U6.3 (+)
- new net: U2.4, U3.5
- new net: U2.11, U2.5, U2.6
- new net: RV1.2, U5.2 (-)
- new net: U3.3, U3.6
- new net: R10.1, U3.4
- new net: D5.2 (A), R17.1
- new net +12V: C3.1, D1.1 (K), K1.2, U1.1 (VI)
- new net +5V: C1.1, C2.1, C4.1, C5.1, C6.1, C7.1, C8.1, C9.1, J4.3 (Pin_3), J6.3 (Pin_3), R13.1, R16.1, R19.2, R7.2, RV1.1, RV2.1, RV3.1, RV4.1, U1.3 (VO), U2.14 (VDD), U3.14 (VDD), U4.8 (Vdd), U5.8 (Vdd), U6.8 (Vdd)
- new net BPSSIG: J4.2 (Pin_2), R7.1, U5.3 (+), U6.2 (-)
- new net GND: C1.2, C10.2, C11.2, C2.2, C3.2, C4.2, C5.2, C6.2, C7.2, C8.2, C9.2, D2.1 (K), D5.1 (K), D6.1 (K), D7.1 (K), J4.1 (Pin_1), J6.1 (Pin_1), Q1.3 (S), R1.2, R15.2, R18.2, R2.2, R3.2, R4.2, R5.2, R6.2, RV1.3, RV2.3, RV3.3, RV4.3, U1.2 (GND), U2.7 (VSS), U3.7 (VSS), U4.4 (Vss), U5.4 (Vss), U6.4 (Vss)
- new net Shutdown1: J5.3 (Pin_3), K1.4
- new net Shutdown2: J5.1 (Pin_1), K1.5
- new net TPSSIG: J6.2 (Pin_2), R19.1, U5.6 (-), U6.6 (-)
Other:
- note added: "11s +- 1s delay"
- note added: "430ms +-40ms delay"
- note added: "Above 4.5V"
- note added: "Both sections have to be active to turn on the MOSFET"
- note added: "Both sensors have to be plugged in for the output to be on"
- note added: "Brake pressure sensor KA sensors: ASL-S1003D Replaced with MIPAG1XX050BSAAX"
- note added: "Braking 30 bar threshold voltage"
- note added: "Checks if sensors are unplugged Due to pullups, if no sensor, voltage above 4.5V shutdown if either unplugged Comparator output high if plugged in"
- note added: "Comparator output N: HIGH SD: LOW"
- note added: "Comparator output N: LOW SD: HIGH"
- note added: "Has to discharge slowly though the 56k but can recharge quickly"
- note added: "Make bypass capacitors close to power pins"
- note added: "NAND output N: HIGH SD: LOW"
- note added: "NAND output N: LOW SD: HIGH"
- note added: "NO NC C"
- note added: "NOTE: This means the system will take 10s to turn on initially!!"
- note added: "NOTES: Check Nuclino for location of parts Individual comparators and NAND gates can be swapped if this improves layout considerations N = normal operation SD = shut down operation"
- note added: "Output high when TPS voltage<threshold i.e. over 25%"
- note added: "Output high when over 30 bar braking"
- note added: "Plugged in if signal <4.5 V, then comparator HIGH"
- note added: "Shutdown circuit terminals Connect between C and NO Due to abiguous datasheet, NO and NC are swapped, the previous statement has accounted for that Could swap the connector to the two pin version"
- note added: "TPS 25% threshold voltage"
- note added: "The NAND output will go HIGH as soon as any LOW input is detected, so it responds instantly to shutdown scenario. NAND needs two HIGH inputs for the output to go LOW so the reset signal is delayed by the RC network. This implements the recovery after 10s. Diode is for it to discharge quickly so that it takes the full time to recharge when the over condition is no longer met"
- note added: "The soldermask legend shows the real relay NC and NO positions. As the BSPD versions are measured when the circuit is on, they are flipped. Between the outer two connections of the shutdown circuit connector, it should be open when the circuit is off, and closed when the circuit is active"
- note added: "Throttle position sensor Possibly just a potentiometer such as P10XXAI103KB30 Voltage decreases with higher throttle position"
- note added: "Unused NAND gate"

Commit message: More labels
Connections:
- net Shutdown1 renamed ShutdownC
- net Shutdown2 renamed ShutdownNO
Changed lines of the file:
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@@
     (effects (font (size 1.27 1.27)) (justify left))
   )
-  (hierarchical_label "Shutdown2" (shape input) (at 370.84 115.57 90)
+  (hierarchical_label "ShutdownNO" (shape input) (at 370.84 115.57 90)
     (effects (font (size 1.27 1.27)) (justify left))
   )
@@
     (effects (font (size 1.27 1.27)) (justify left))
   )
-  (hierarchical_label "Shutdown1" (shape input) (at 368.3 120.65 90)
+  (hierarchical_label "ShutdownC" (shape input) (at 368.3 120.65 90)
     (effects (font (size 1.27 1.27)) (justify left))
   )
