File: Loom23/ECU.kicad_sch (KiCad schematic)
At the start: 0 parts

Commit message: Added detailed version of schematic
Other:
- note added: "ECU"
Changed lines of the file:
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@@
 (kicad_sch (version 20211123) (generator eeschema)
   (paper "A4")
+  (polyline (pts (xy 57.15 101.6) (xy 57.15 135.89))
+    (stroke (width 0) (type default) (color 0 0 0 0))
+  )
+  (polyline (pts (xy 57.15 135.89) (xy 149.86 135.89))
+    (stroke (width 0) (type default) (color 0 0 0 0))
+  )
+  (polyline (pts (xy 57.15 101.6) (xy 149.86 101.6))
+    (stroke (width 0) (type default) (color 0 0 0 0))
+  )
+  (polyline (pts (xy 149.86 135.89) (xy 149.86 101.6))
+    (stroke (width 0) (type default) (color 0 0 0 0))
+  )
+  (text "ECU\n\n\n" (at 97.79 137.16 0)
+    (effects (font (size 5 5)) (justify left bottom))
+  )
+  (hierarchical_label "CAN Low (Pin 3)" (shape input) (at 64.77 96.52 90)
+    (effects (font (size 1.27 1.27)) (justify left))
+  )
+  (hierarchical_label "INJECTOR 2 (Pin 10)" (shape input) (at 82.55 96.52 90)
+    (effects (font (size 1.27 1.27)) (justify left))
+  )
+  (hierarchical_label "TACH OUTPUT (Pin 35)" (shape input) (at 146.05 96.52 90)
+    (effects (font (size 1.27 1.27)) (justify left))
+  )
+  (hierarchical_label "BOOTLOADER (Pin 15)" (shape input) (at 95.25 96.52 90)
+    (effects (font (size 1.27 1.27)) (justify left))
+  )
+  (hierarchical_label "Spare Input 1 (Pin 29)" (shape input) (at 130.81 96.52 90)
+    (effects (font (size 1.27 1.27)) (justify left))
+  )
+  (hierarchical_label "FUEL PUMP (Pin 8)" (shape input) (at 77.47 96.52 90)
+    (effects (font (size 1.27 1.27)) (justify left))
+  )
+  (hierarchical_label "ECU12V (Pin 1)" (shape input) (at 59.69 96.52 90)
+    (effects (font (size 1.27 1.27)) (justify left))
+  )
+  (hierarchical_label "VRIN2+ (Pin 4)" (shape input) (at 67.31 96.52 90)
+    (effects (font (size 1.27 1.27)) (justify left))
+  )
+  (hierarchical_label "OPTOIN- (Pin 31)" (shape input) (at 135.89 96.52 90)
+    (effects (font (size 1.27 1.27)) (justify left))
+  )
+  (hierarchical_label "OPTOIN+ (Pin 30)" (shape input) (at 133.35 96.52 90)
+    (effects (font (size 1.27 1.27)) (justify left))
+  )
+  (hierarchical_label "MAP (Pin 24)" (shape input) (at 118.11 96.52 90)
+    (effects (font (size 1.27 1.27)) (justify left))
+  )
+  (hierarchical_label "INJECTOR 1 (Pin 9)" (shape input) (at 80.01 96.52 90)
+    (effects (font (size 1.27 1.27)) (justify left))
+  )
+  (hierarchical_label "GROUND (Pin 23)" (shape input) (at 115.57 96.52 90)
+    (effects (font (size 1.27 1.27)) (justify left))
+  )
+  (hierarchical_label "IGNITION OUTPUT 1 (Pin 12)" (shape input) (at 87.63 96.52 90)
+    (effects (font (size 1.27 1.27)) (justify left))
+  )
+  (hierarchical_label "CAN High (Pin 2)" (shape input) (at 62.23 96.52 90)
+    (effects (font (size 1.27 1.27)) (justify left))
+  )
+  (hierarchical_label "TPS (Pin 27)" (shape input) (at 125.73 96.52 90)
+    (effects (font (size 1.27 1.27)) (justify left))
+  )
+  (hierarchical_label "IAT (Pin 26)" (shape input) (at 123.19 96.52 90)
+    (effects (font (size 1.27 1.27)) (justify left))
+  )
+  (hierarchical_label "FIDLE (Pin 7)" (shape input) (at 74.93 96.52 90)
+    (effects (font (size 1.27 1.27)) (justify left))
+  )
+  (hierarchical_label "Spare Input 2 (Pin 5)" (shape input) (at 69.85 96.52 90)
+    (effects (font (size 1.27 1.27)) (justify left))
+  )
+  (hierarchical_label "GROUND (Pin 22)" (shape input) (at 113.03 96.52 90)
+    (effects (font (size 1.27 1.27)) (justify left))
+  )
+  (hierarchical_label "WARM-UP LED (Pin 17)" (shape input) (at 100.33 96.52 90)
+    (effects (font (size 1.27 1.27)) (justify left))
+  )
+  (hierarchical_label "VRIN- (Pin 33)" (shape input) (at 140.97 96.52 90)
+    (effects (font (size 1.27 1.27)) (justify left))
+  )
+  (hierarchical_label "Serial Tx (Pin 14)" (shape input) (at 92.71 96.52 90)
+    (effects (font (size 1.27 1.27)) (justify left))
+  )
+  (hierarchical_label "VR2IN- (Pin 21)" (shape input) (at 110.49 96.52 90)
+    (effects (font (size 1.27 1.27)) (justify left))
+  )
+  (hierarchical_label "CLT (Pin 25)" (shape input) (at 120.65 96.52 90)
+    (effects (font (size 1.27 1.27)) (justify left))
+  )
+  (hierarchical_label "SENSOR GROUND (Pin 20)" (shape input) (at 107.95 96.52 90)
+    (effects (font (size 1.27 1.27)) (justify left))
+  )
+  (hierarchical_label "Serial Rx (Pin 13)" (shape input) (at 90.17 96.52 90)
+    (effects (font (size 1.27 1.27)) (justify left))
+  )
+  (hierarchical_label "VRIN1+ (Pin 32)" (shape input) (at 138.43 96.52 90)
+    (effects (font (size 1.27 1.27)) (justify left))
+  )
+  (hierarchical_label "2ND SENSOR GROUND (Pin 18)" (shape input) (at 102.87 96.52 90)
+    (effects (font (size 1.27 1.27)) (justify left))
+  )
+  (hierarchical_label "Vref (Pin 28)" (shape input) (at 128.27 96.52 90)
+    (effects (font (size 1.27 1.27)) (justify left))
+  )
+  (hierarchical_label "ACCEL LED (Pin 16)" (shape input) (at 97.79 96.52 90)
+    (effects (font (size 1.27 1.27)) (justify left))
+  )
+  (hierarchical_label "O2 (Pin 34)" (shape input) (at 143.51 96.52 90)
+    (effects (font (size 1.27 1.27)) (justify left))
+  )
+  (hierarchical_label "Flex Fuel (Pin 6)" (shape input) (at 72.39 96.52 90)
+    (effects (font (size 1.27 1.27)) (justify left))
+  )
+  (hierarchical_label "SERIAL GROUND (Pin 19)" (shape input) (at 105.41 96.52 90)
+    (effects (font (size 1.27 1.27)) (justify left))
+  )
+  (hierarchical_label "IGNITION OUTPUT 2 (Pin 11)" (shape input) (at 85.09 96.52 90)
+    (effects (font (size 1.27 1.27)) (justify left))
+  )
 )
