File: Loom23/MAP.kicad_sch (KiCad schematic)
At the start: 0 parts

Commit message: Added detailed version of schematic
Parts:
- added RV?: (no value), symbol Device:R_Potentiometer
Connections:
- new net +5V (Pin 3): RV?.1
- new net MAPSIG (Pin 2): RV?.2
- new net SENGND (Pin 1): RV?.3
Changed lines of the file:
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@@
 (kicad_sch (version 20211123) (generator eeschema)
   (paper "A4")
+  (wire (pts (xy 163.83 95.25) (xy 163.83 99.06))
+    (stroke (width 0) (type default) (color 0 0 0 0))
+  )
+  (wire (pts (xy 152.4 91.44) (xy 160.02 91.44))
+    (stroke (width 0) (type default) (color 0 0 0 0))
+  )
+  (wire (pts (xy 167.64 91.44) (xy 172.72 91.44))
+    (stroke (width 0) (type default) (color 0 0 0 0))
+  )
+  (hierarchical_label "+5V (Pin 3)" (shape input) (at 172.72 91.44 0)
+    (effects (font (size 1.27 1.27)) (justify left))
+  )
+  (hierarchical_label "MAPSIG (Pin 2)" (shape input) (at 163.83 99.06 270)
+    (effects (font (size 1.27 1.27)) (justify right))
+  )
+  (hierarchical_label "SENGND (Pin 1)" (shape input) (at 152.4 91.44 180)
+    (effects (font (size 1.27 1.27)) (justify right))
+  )
+  (symbol (lib_id "Device:R_Potentiometer") (at 163.83 91.44 270) (unit 1)
+    (in_bom yes) (on_board yes) (fields_autoplaced)
+    (property "Reference" "RV?" (id 0) (at 163.83 85.09 90))
+    (property "Value" "" (id 1) (at 163.83 87.63 90))
+    (property "Footprint" "" (id 2) (at 163.83 91.44 0)
+      (effects (font (size 1.27 1.27)) hide)
+    )
+    (property "Datasheet" "~" (id 3) (at 163.83 91.44 0)
+      (effects (font (size 1.27 1.27)) hide)
+    )
+    (pin "1")
+    (pin "2")
+    (pin "3")
+  )
 )

Commit message: Signed-off-by: fst29 <fst29@cam.ac.uk>
Parts:
- RV?: value (none) -> R_Potentiometer
Changed lines of the file:
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@@
     (in_bom yes) (on_board yes) (fields_autoplaced)
     (property "Reference" "RV?" (id 0) (at 163.83 85.09 90))
-    (property "Value" "" (id 1) (at 163.83 87.63 90))
+    (property "Value" "R_Potentiometer" (id 1) (at 163.83 87.63 90))
     (property "Footprint" "" (id 2) (at 163.83 91.44 0)
       (effects (font (size 1.27 1.27)) hide)
