File: Loom23/TPS (ECU).kicad_sch (KiCad schematic)
At the start: 0 parts

Commit message: Added detailed version of schematic
Parts:
- added RV?: R_Potentiometer, symbol Device:R_Potentiometer
Connections:
- new net +5V (Pin C): RV?.1
- new net SENGND (Pin A): RV?.3
- new net TSP(ECU) Signal (Pin B): RV?.2
Changed lines of the file:
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@@
 (kicad_sch (version 20211123) (generator eeschema)
   (paper "A4")
+  (wire (pts (xy 100.33 95.25) (xy 107.95 95.25))
+    (stroke (width 0) (type default) (color 0 0 0 0))
+  )
+  (wire (pts (xy 111.76 99.06) (xy 111.76 101.6))
+    (stroke (width 0) (type default) (color 0 0 0 0))
+  )
+  (wire (pts (xy 115.57 95.25) (xy 118.11 95.25))
+    (stroke (width 0) (type default) (color 0 0 0 0))
+  )
+  (hierarchical_label "SENGND (Pin A)" (shape input) (at 100.33 95.25 180)
+    (effects (font (size 1.27 1.27)) (justify right))
+  )
+  (hierarchical_label "+5V (Pin C)" (shape input) (at 118.11 95.25 0)
+    (effects (font (size 1.27 1.27)) (justify left))
+  )
+  (hierarchical_label "TSP(ECU) Signal (Pin B)" (shape input) (at 111.76 101.6 270)
+    (effects (font (size 1.27 1.27)) (justify right))
+  )
+  (symbol (lib_id "Device:R_Potentiometer") (at 111.76 95.25 270) (unit 1)
+    (in_bom yes) (on_board yes) (fields_autoplaced)
+    (property "Reference" "RV?" (id 0) (at 111.76 88.9 90))
+    (property "Value" "R_Potentiometer" (id 1) (at 111.76 91.44 90))
+    (property "Footprint" "" (id 2) (at 111.76 95.25 0)
+      (effects (font (size 1.27 1.27)) hide)
+    )
+    (property "Datasheet" "~" (id 3) (at 111.76 95.25 0)
+      (effects (font (size 1.27 1.27)) hide)
+    )
+    (pin "1")
+    (pin "2")
+    (pin "3")
+  )
 )
