File: Loom23/ignition.kicad_sch (KiCad schematic)
At the start: 0 parts

Commit message: Added fuel pump, TPS(BSPD), BPS.
Other:
- note added: "Connector types?"
- note added: "High side to relay"
- note added: "Ignition controller URO Parts 4D0905351"
- note added: "Needs good ground connection"
- note removed: "Ignition controller Type TBC"
Changed lines of the file:
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@@
     (stroke (width 0) (type default) (color 0 0 0 0))
   )
-  (text "Ignition controller\nType TBC" (at 101.6 97.79 0)
+  (text "Ignition controller\nURO Parts 4D0905351" (at 99.06 104.14 0)
     (effects (font (size 1.27 1.27)) (justify left bottom))
   )
@@
     (effects (font (size 1.27 1.27)) (justify left bottom))
   )
+  (text "High side to relay" (at 252.73 54.61 0)
+    (effects (font (size 1.27 1.27)) (justify left bottom))
+  )
   (text "Spark plug3" (at 208.28 93.98 0)
     (effects (font (size 1.27 1.27)) (justify left bottom))
   )
+  (text "Connector types?\n" (at 101.6 119.38 0)
+    (effects (font (size 1.27 1.27)) (justify left bottom))
+  )
+  (text "Needs good ground connection" (at 247.65 77.47 0)
+    (effects (font (size 1.27 1.27)) (justify left bottom))
+  )
