File: Loom23/Loom23_detailed.kicad_sch (KiCad schematic)
At the start: 7 parts

Commit message: Included BSPD and started adding labels
Parts:
- gave numbers to parts that had none: 5
Connections:
- net BSPD/Shutdown2: now reaches SW_Inertia.1
- net Starter relay/+12V: now reaches F?.1, SW_LVMS.1
- no-connect marks 4 -> 7
Other:
- removed sheet Ride height sensors (4x)
- sheet BSPD ports: added +12V, BPS+5V, BPSGND, BPSSIG, GND, Shutdown1, Shutdown2, TPS+5V, TPSGND, TPSSIG; removed none
- sheet Starter motor ports: added none; removed GND
- sheet Starter relay ports: added +12V, GND, Starter Signal, StarterPower; removed none
- note added: "Confirm spark-ECU Pairing"
- note removed: "Confirm pairing"
- note removed: "Confirm spark order"

Commit message: More labels
Connections:
- net Shutdown6: now reaches SW_BOTS.1, SW_Inertia.2
- net Shutdown2: now reaches SW_LEStop.1, SW_REStop.2
- net BSPD/Shutdown2 renamed Shutdown5
- net Dash switches/Shutdown 1 renamed Shutdown3
- net Fusebox/From LVMS renamed LVMS+12V
- net Relaybox/Shutdown signal renamed Shutdown7
Other:
- sheet BSPD ports: added ShutdownC, ShutdownNO; removed Shutdown1, Shutdown2

Commit message: Finished wire labels
Other:
- sheet Dash Break-out-board ports: added DASH GND; removed DASH GNG
- note added: "Ethernet cable"

Commit message: Created a spreadsheet with all the wires
Connections:
- net Starter relay/+12V renamed BATT
Other:
- note added: "Within 100mm of the +ve terminal"
Changed lines of the file:
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@@
+    (effects (font (size 1.27 1.27)) (justify left bottom))
+  )
+  (text "Within 100mm of the +ve terminal\n" (at 467.36 85.09 0)
     (effects (font (size 1.27 1.27)) (justify left bottom))
   )
@@
     (effects (font (size 1.27 1.27)) (justify left bottom))
   )
+  (label "STARTERRELAY" (at 381.635 62.23 0)
+    (effects (font (size 0.5 0.5)) (justify left bottom))
+  )
   (label "LAMBDA+12V" (at 378.46 149.86 0)
     (effects (font (size 0.6 0.6)) (justify left bottom))
@@
     (effects (font (size 1.27 1.27)) (justify left bottom))
   )
-  (label "SPK " (at 417.83 204.47 0)
+  (label "SPK" (at 417.83 204.47 0)
     (effects (font (size 1.27 1.27)) (justify left bottom))
   )
@@
     (effects (font (size 1.27 1.27)) (justify left bottom))
   )
+  (label "BATT" (at 449.58 73.66 0)
+    (effects (font (size 1.27 1.27)) (justify left bottom))
+  )
   (label "FANPWR" (at 212.09 143.51 0)
     (effects (font (size 0.5 0.5)) (justify left bottom))
@@
     (effects (font (size 1.27 1.27)) (justify left bottom))
   )
-  (label "SPK" (at 212.09 148.59 0)
+  (label "SPK R-F" (at 212.09 148.59 0)
     (effects (font (size 0.5 0.5)) (justify left bottom))
   )
@@
     (effects (font (size 0.6 0.6)) (justify left bottom))
   )
-  (label "SPK " (at 289.56 127 90)
-    (effects (font (size 1.27 1.27)) (justify left bottom))
-  )
-  (label "INJPWR" (at 300.99 100.33 90)
-    (effects (font (size 1.27 1.27)) (justify left bottom))
+  (label "SPK" (at 289.56 127 90)
+    (effects (font (size 1.27 1.27)) (justify left bottom))
+  )
+  (label "BATT" (at 461.01 80.645 0)
+    (effects (font (size 1.27 1.27)) (justify left bottom))
+  )
+  (label "INJPWR F-R" (at 300.99 100.33 90)
+    (effects (font (size 1.27 1.27)) (justify left bottom))
+  )
+  (label "STARTERRELAY" (at 461.01 68.58 90)
+    (effects (font (size 0.5 0.5)) (justify left bottom))
   )
   (label "MAPSIG" (at 63.5 218.44 0)
     (effects (font (size 1.27 1.27)) (justify left bottom))
   )
-  (label "INJPWR" (at 212.09 146.05 0)
+  (label "INJPWR F-R" (at 212.09 146.05 0)
     (effects (font (size 0.5 0.5)) (justify left bottom))
   )
@@
     (effects (font (size 1.27 1.27)) (justify right bottom))
   )
-  (label "FPPWR" (at 212.09 139.7 0)
+  (label "FPPWR R-F" (at 212.09 139.7 0)
     (effects (font (size 0.5 0.5)) (justify left bottom))
   )
@@
     (effects (font (size 1.27 1.27)) (justify right bottom))
   )
+  (label "OPTOIN-" (at 63.5 236.22 0)
+    (effects (font (size 1.27 1.27)) (justify left bottom))
+  )
   (label "INJ2,4LOW" (at 63.5 182.88 0)
     (effects (font (size 1.27 1.27)) (justify left bottom))
   )
+  (label "SI2" (at 62.865 170.18 0)
+    (effects (font (size 1.1 1.1)) (justify left bottom))
+  )
   (label "IATSIG" (at 384.81 124.46 180)
     (effects (font (size 0.4 0.4)) (justify right bottom))
@@
     (effects (font (size 1.27 1.27)) (justify left bottom))
   )
-  (label "SPK" (at 292.1 99.06 90)
+  (label "SPK R-F" (at 292.1 99.06 90)
     (effects (font (size 1.27 1.27)) (justify left bottom))
   )
@@
     (effects (font (size 1.27 1.27)) (justify left bottom))
   )
-  (label "FPPWR" (at 309.88 99.06 90)
+  (label "FPPWR R-F" (at 309.88 99.06 90)
     (effects (font (size 1.27 1.27)) (justify left bottom))
   )
@@
     (effects (font (size 1.27 1.27)) (justify left bottom))
   )
+  (label "OPTOIN+" (at 63.5 233.68 0)
+    (effects (font (size 1.27 1.27)) (justify left bottom))
+  )
   (label "TPS2+5V" (at 205.74 184.15 0)
     (effects (font (size 1.27 1.27)) (justify left bottom))
@@
     (effects (font (size 0.6 0.6)) (justify left bottom))
   )
+  (label "SI1" (at 63.5 231.14 0)
+    (effects (font (size 1.27 1.27)) (justify left bottom))
+  )
   (label "ECU+12V" (at 63.5 157.48 90)

Commit message: Added engine speed sensor, fixed INJ and IGN connections
Connections:
- no-connect marks 7 -> 8
Other:
- added sheet Engine speed sensor (EngineSpeed.kicad_sch)
- note added: "Assuming cylinder 1 is on the left High impedance injectors, no extra resistors needed."
- note removed: "Confirm spark-ECU Pairing"
- note removed: "Pairing and connector type TBC High impedance injectors, no extra resistors needed."

Commit message: Added colours
Other:
- note added: "Not finalised yet"
