File: Loom23/Relaybox.kicad_sch (KiCad schematic)
At the start: 4 parts

Commit message: Changes made to fusebox, relayboard and camsensor
Parts:
- added K?: ADW11, Relay_THT:Relay_1P1T_NO_10x24x18.8mm_Panasonic_ADW11xxxxW_THT, symbol Relay:ADW11
Connections:
- net +12V: now also K?.1
- net Fuel pump enable (ECU): now also K?.6
- net RelayedSpark: now also K?.5; no longer K?.5
- new net: K?.3, K?.5
Other:
- moved on the sheet: K?
Changed lines of the file:
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@@
 (kicad_sch (version 20211123) (generator eeschema)
   (paper "A4")
+  (junction (at 101.6 67.31) (diameter 0) (color 0 0 0 0)
+  )
+  (junction (at 99.06 48.26) (diameter 0) (color 0 0 0 0)
+  )
   (junction (at 99.06 74.93) (diameter 0) (color 0 0 0 0)
   )
   (junction (at 114.3 127) (diameter 0) (color 0 0 0 0)
   )
-  (junction (at 96.52 45.72) (diameter 0) (color 0 0 0 0)
+  (junction (at 96.52 22.86) (diameter 0) (color 0 0 0 0)
   )
   (junction (at 99.06 100.33) (diameter 0) (color 0 0 0 0)
   )
-  (junction (at 99.06 43.18) (diameter 0) (color 0 0 0 0)
+  (junction (at 99.06 20.32) (diameter 0) (color 0 0 0 0)
   )
   (junction (at 96.52 77.47) (diameter 0) (color 0 0 0 0)
   )
-  (wire (pts (xy 96.52 43.18) (xy 96.52 45.72))
-    (stroke (width 0) (type default) (color 0 0 0 0))
-  )
-  (wire (pts (xy 99.06 43.18) (xy 99.06 74.93))
-    (stroke (width 0) (type default) (color 0 0 0 0))
-  )
-  (wire (pts (xy 125.73 60.96) (xy 147.32 60.96))
-    (stroke (width 0) (type default) (color 0 0 0 0))
-  )
-  (wire (pts (xy 96.52 45.72) (xy 96.52 77.47))
-    (stroke (width 0) (type default) (color 0 0 0 0))
-  )
-  (wire (pts (xy 86.36 92.71) (xy 114.3 92.71))
+  (wire (pts (xy 115.57 63.5) (xy 115.57 67.31))
+    (stroke (width 0) (type default) (color 0 0 0 0))
+  )
+  (wire (pts (xy 96.52 20.32) (xy 96.52 22.86))
+    (stroke (width 0) (type default) (color 0 0 0 0))
+  )
+  (wire (pts (xy 125.73 63.5) (xy 147.32 63.5))
+    (stroke (width 0) (type default) (color 0 0 0 0))
+  )
+  (wire (pts (xy 101.6 92.71) (xy 114.3 92.71))
+    (stroke (width 0) (type default) (color 0 0 0 0))
+  )
+  (wire (pts (xy 86.36 67.31) (xy 101.6 67.31))
     (stroke (width 0) (type default) (color 0 0 0 0))
   )
@@
     (stroke (width 0) (type default) (color 0 0 0 0))
   )
-  (wire (pts (xy 99.06 40.64) (xy 99.06 43.18))
+  (wire (pts (xy 99.06 17.78) (xy 99.06 20.32))
     (stroke (width 0) (type default) (color 0 0 0 0))
   )
@@
     (stroke (width 0) (type default) (color 0 0 0 0))
   )
+  (wire (pts (xy 115.57 67.31) (xy 101.6 67.31))
+    (stroke (width 0) (type default) (color 0 0 0 0))
+  )
   (wire (pts (xy 96.52 102.87) (xy 114.3 102.87))
     (stroke (width 0) (type default) (color 0 0 0 0))
   )
-  (wire (pts (xy 86.36 60.96) (xy 115.57 60.96))
+  (wire (pts (xy 86.36 38.1) (xy 115.57 38.1))
     (stroke (width 0) (type default) (color 0 0 0 0))
   )
@@
     (stroke (width 0) (type default) (color 0 0 0 0))
   )
+  (wire (pts (xy 99.06 20.32) (xy 99.06 48.26))
+    (stroke (width 0) (type default) (color 0 0 0 0))
+  )
   (wire (pts (xy 99.06 74.93) (xy 99.06 100.33))
     (stroke (width 0) (type default) (color 0 0 0 0))
   )
-  (wire (pts (xy 128.27 45.72) (xy 128.27 43.18))
+  (wire (pts (xy 96.52 22.86) (xy 96.52 77.47))
+    (stroke (width 0) (type default) (color 0 0 0 0))
+  )
+  (wire (pts (xy 128.27 38.1) (xy 128.27 48.26))
+    (stroke (width 0) (type default) (color 0 0 0 0))
+  )
+  (wire (pts (xy 128.27 22.86) (xy 128.27 20.32))
     (stroke (width 0) (type default) (color 0 0 0 0))
   )
@@
     (stroke (width 0) (type default) (color 0 0 0 0))
   )
-  (wire (pts (xy 115.57 45.72) (xy 96.52 45.72))
+  (wire (pts (xy 115.57 22.86) (xy 96.52 22.86))
     (stroke (width 0) (type default) (color 0 0 0 0))
   )
@@
     (stroke (width 0) (type default) (color 0 0 0 0))
   )
-  (wire (pts (xy 86.36 43.18) (xy 96.52 43.18))
-    (stroke (width 0) (type default) (color 0 0 0 0))
-  )
-  (wire (pts (xy 86.36 40.64) (xy 99.06 40.64))
+  (wire (pts (xy 86.36 20.32) (xy 96.52 20.32))
+    (stroke (width 0) (type default) (color 0 0 0 0))
+  )
+  (wire (pts (xy 99.06 48.26) (xy 115.57 48.26))
+    (stroke (width 0) (type default) (color 0 0 0 0))
+  )
+  (wire (pts (xy 125.73 38.1) (xy 128.27 38.1))
+    (stroke (width 0) (type default) (color 0 0 0 0))
+  )
+  (wire (pts (xy 101.6 67.31) (xy 101.6 92.71))
+    (stroke (width 0) (type default) (color 0 0 0 0))
+  )
+  (wire (pts (xy 86.36 17.78) (xy 99.06 17.78))
     (stroke (width 0) (type default) (color 0 0 0 0))
   )
@@
     (stroke (width 0) (type default) (color 0 0 0 0))
   )
-  (wire (pts (xy 99.06 43.18) (xy 128.27 43.18))
+  (wire (pts (xy 99.06 20.32) (xy 128.27 20.32))
     (stroke (width 0) (type default) (color 0 0 0 0))
   )
@@
     (stroke (width 0) (type default) (color 0 0 0 0))
   )
+  (wire (pts (xy 99.06 48.26) (xy 99.06 74.93))
+    (stroke (width 0) (type default) (color 0 0 0 0))
+  )
   (hierarchical_label "Relayed Fan" (shape input) (at 147.32 142.24 0)
     (effects (font (size 1.27 1.27)) (justify left))
@@
     (effects (font (size 1.27 1.27)) (justify left))
   )
-  (hierarchical_label "Fuel pump enable (ECU)" (shape input) (at 86.36 92.71 180)
-    (effects (font (size 1.27 1.27)) (justify right))
-  )
-  (hierarchical_label "Paddle shifter" (shape input) (at 86.36 60.96 180)
-    (effects (font (size 1.27 1.27)) (justify right))
-  )
-  (hierarchical_label "RelayedSpark" (shape input) (at 147.32 60.96 0)
+  (hierarchical_label "Fuel pump enable (ECU)" (shape input) (at 86.36 67.31 180)
+    (effects (font (size 1.27 1.27)) (justify right))
+  )
+  (hierarchical_label "Paddle shifter" (shape input) (at 86.36 38.1 180)
+    (effects (font (size 1.27 1.27)) (justify right))
+  )
+  (hierarchical_label "RelayedSpark" (shape input) (at 147.32 63.5 0)
     (effects (font (size 1.27 1.27)) (justify left))
   )
@@
     (effects (font (size 1.27 1.27)) (justify right))
   )
-  (hierarchical_label "+12V" (shape input) (at 86.36 40.64 180)
-    (effects (font (size 1.27 1.27)) (justify right))
-  )
-  (hierarchical_label "Shutdown signal" (shape input) (at 86.36 43.18 180)
+  (hierarchical_label "+12V" (shape input) (at 86.36 17.78 180)
+    (effects (font (size 1.27 1.27)) (justify right))
+  )
+  (hierarchical_label "Shutdown signal" (shape input) (at 86.36 20.32 180)
     (effects (font (size 1.27 1.27)) (justify right))
   )
@@
     (pin "6")
   )
+  (symbol (lib_id "Relay:ADW11") (at 120.65 55.88 0) (unit 1)
+    (in_bom yes) (on_board yes) (fields_autoplaced)
+    (property "Reference" "K?" (id 0) (at 132.08 54.6099 0)
+      (effects (font (size 1.27 1.27)) (justify left))
+    )
+    (property "Value" "ADW11" (id 1) (at 132.08 57.1499 0)
+      (effects (font (size 1.27 1.27)) (justify left))
+    )
+    (property "Footprint" "Relay_THT:Relay_1P1T_NO_10x24x18.8mm_Panasonic_ADW11xxxxW_THT" (id 2) (at 154.305 57.15 0)
+      (effects (font (size 1.27 1.27)) hide)
+    )
+    (property "Datasheet" "https://www.panasonic-electric-works.com/pew/es/downloads/ds_dw_hl_en.pdf" (id 3) (at 120.65 55.88 0)
+      (effects (font (size 1.27 1.27)) hide)
+    )
+    (pin "1")
+    (pin "3")
+    (pin "5")
+    (pin "6")
+  )
   (symbol (lib_id "Relay:ADW11") (at 119.38 85.09 0) (unit 1)
     (in_bom yes) (on_board yes) (fields_autoplaced)
@@
     (pin "6")
   )
-  (symbol (lib_id "Relay:ADW11") (at 120.65 53.34 0) (unit 1)
-    (in_bom yes) (on_board yes) (fields_autoplaced)
-    (property "Reference" "K?" (id 0) (at 132.08 52.0699 0)
-      (effects (font (size 1.27 1.27)) (justify left))
-    )
-    (property "Value" "ADW11" (id 1) (at 132.08 54.6099 0)
-      (effects (font (size 1.27 1.27)) (justify left))
-    )
-    (property "Footprint" "Relay_THT:Relay_1P1T_NO_10x24x18.8mm_Panasonic_ADW11xxxxW_THT" (id 2) (at 154.305 54.61 0)
-      (effects (font (size 1.27 1.27)) hide)
-    )
-    (property "Datasheet" "https://www.panasonic-electric-works.com/pew/es/downloads/ds_dw_hl_en.pdf" (id 3) (at 120.65 53.34 0)
-      (effects (font (size 1.27 1.27)) hide)
-    )
+  (symbol (lib_id "Relay:ADW11") (at 120.65 30.48 0) (unit 1)
+    (in_bom yes) (on_board yes) (fields_autoplaced)
+    (property "Reference" "K?" (id 0) (at 132.08 29.2099 0)
+      (effects (font (size 1.27 1.27)) (justify left))
+    )
+    (property "Value" "ADW11" (id 1) (at 132.08 31.7499 0)
+      (effects (font (size 1.27 1.27)) (justify left))
+    )
+    (property "Footprint" "Relay_THT:Relay_1P1T_NO_10x24x18.8mm_Panasonic_ADW11xxxxW_THT" (id 2) (at 154.305 31.75 0)
+      (effects (font (size 1.27 1.27)) hide)
+    )
+    (property "Datasheet" "https://www.panasonic-electric-works.com/pew/es/downloads/ds_dw_hl_en.pdf" (id 3) (at 120.65 30.48 0)
+      (effects (font (size 1.27 1.27)) hide)
+    )

Commit message: Changed labels to match old wires
Connections:
- net Fan signal renamed FANSIG
- net Fuel pump enable (ECU) renamed FPSIG
- net Paddle shifter renamed Sparkstop
- net Relayed Fan renamed FANPWR R-F
- net Relayed Injectors renamed INJPWR R-F
- net Relayed fuel pump renamed FPPWR R-F
- net RelayedSpark renamed SPK R-F
- net Shutdown signal renamed Shutdown
Other:
- note added: "Connector label: Relays Connector type: Deutsch DT 6 pin"
- note added: "Connector label: Relays-Fuses Connector type: TBD"
- note added: "Pin1 Pin2 Pin3 Pin4"
- note added: "Pin1 Pin2 Pin3 Pin4 Pin5 Pin6 Not connected"
Changed lines of the file:
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@@
     (stroke (width 0) (type default) (color 0 0 0 0))
   )
-  (hierarchical_label "Relayed Fan" (shape input) (at 147.32 142.24 0)
+  (text "Connector label: Relays-Fuses\nConnector type: TBD\n"
+    (at 210.312 51.562 0)
+    (effects (font (size 1.27 1.27)) (justify left bottom))
+  )
+  (text "Connector label: Relays\nConnector type: Deutsch DT 6 pin\n\n"
+    (at 22.606 38.862 0)
+    (effects (font (size 1.27 1.27)) (justify left bottom))
+  )
+  (text "Pin1\nPin2\nPin3\nPin4\nPin5\nPin6 Not connected\n" (at 22.606 52.324 0)
+    (effects (font (size 1.27 1.27)) (justify left bottom))
+  )
+  (text "Pin1\nPin2\nPin3\nPin4\n\n\n" (at 210.312 65.024 0)
+    (effects (font (size 1.27 1.27)) (justify left bottom))
+  )
+  (hierarchical_label "FANPWR R-F" (shape input) (at 147.32 142.24 0)
     (effects (font (size 1.27 1.27)) (justify left))
   )
-  (hierarchical_label "Relayed Injectors" (shape input) (at 147.32 118.11 0)
+  (hierarchical_label "INJPWR R-F" (shape input) (at 147.32 118.11 0)
     (effects (font (size 1.27 1.27)) (justify left))
   )
-  (hierarchical_label "Fuel pump enable (ECU)" (shape input) (at 86.36 67.31 180)
+  (hierarchical_label "FPSIG" (shape input) (at 86.36 67.31 180)
     (effects (font (size 1.27 1.27)) (justify right))
   )
-  (hierarchical_label "Paddle shifter" (shape input) (at 86.36 38.1 180)
+  (hierarchical_label "Sparkstop" (shape input) (at 86.36 38.1 180)
     (effects (font (size 1.27 1.27)) (justify right))
   )
-  (hierarchical_label "RelayedSpark" (shape input) (at 147.32 63.5 0)
+  (hierarchical_label "FPPWR R-F" (shape input) (at 215.646 55.372 0)
     (effects (font (size 1.27 1.27)) (justify left))
   )
-  (hierarchical_label "Relayed fuel pump" (shape input) (at 147.32 92.71 0)
+  (hierarchical_label "FPSIG" (shape input) (at 27.94 46.482 0)
     (effects (font (size 1.27 1.27)) (justify left))
   )
-  (hierarchical_label "Fan signal" (shape input) (at 85.09 142.24 180)
+  (hierarchical_label "SPK R-F" (shape input) (at 147.32 63.5 0)
+    (effects (font (size 1.27 1.27)) (justify left))
+  )
+  (hierarchical_label "FPPWR R-F" (shape input) (at 147.32 92.71 0)
+    (effects (font (size 1.27 1.27)) (justify left))
+  )
+  (hierarchical_label "FANSIG" (shape input) (at 85.09 142.24 180)
     (effects (font (size 1.27 1.27)) (justify right))
+  )
+  (hierarchical_label "FANSIG" (shape input) (at 27.94 48.768 0)
+    (effects (font (size 1.27 1.27)) (justify left))
+  )
+  (hierarchical_label "+12V" (shape input) (at 27.94 40.64 0)
+    (effects (font (size 1.27 1.27)) (justify left))
+  )
+  (hierarchical_label "Sparkstop" (shape input) (at 27.94 44.704 0)
+    (effects (font (size 1.27 1.27)) (justify left))
+  )
+  (hierarchical_label "SPK R-F" (shape input) (at 215.646 53.34 0)
+    (effects (font (size 1.27 1.27)) (justify left))
   )
   (hierarchical_label "+12V" (shape input) (at 86.36 17.78 180)
     (effects (font (size 1.27 1.27)) (justify right))
   )
-  (hierarchical_label "Shutdown signal" (shape input) (at 86.36 20.32 180)
+  (hierarchical_label "FANPWR R-F" (shape input) (at 215.646 59.182 0)
+    (effects (font (size 1.27 1.27)) (justify left))
+  )
+  (hierarchical_label "Shutdown" (shape input) (at 86.36 20.32 180)
     (effects (font (size 1.27 1.27)) (justify right))
   )
+  (hierarchical_label "INJPWR R-F" (shape input) (at 215.646 57.404 0)
+    (effects (font (size 1.27 1.27)) (justify left))
+  )
+  (hierarchical_label "Shutdown" (shape input) (at 27.94 42.672 0)
+    (effects (font (size 1.27 1.27)) (justify left))
+  )
   (hierarchical_label "GND" (shape input) (at 86.36 118.11 180)
