File: Loom23/Dash switches.kicad_sch (KiCad schematic)
At the start: 0 parts

Commit message: Added dash switches and crank sensor.
Parts:
- added SW? (x2): SW_SPST, symbol Switch:SW_SPST
- added SW?: SW_MEC_5G, symbol Switch:SW_MEC_5G
Connections:
- new net GND: SW?.1 (A), SW?.1 (A), SW?.2 (A)
- new net Launch control: SW?.2 (B)
- new net Shutdown 1: SW?.1 (A)
- new net Shutdown2: SW?.2 (B)
- new net StarterSignal: SW?.3 (B), SW?.4 (B)
Other:
- note added: "Cockpit EStop"
- note added: "Launch control"
- note added: "Starter button"
Changed lines of the file:
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@@
 (kicad_sch (version 20211123) (generator eeschema)
   (paper "A4")
+  (junction (at 163.83 80.01) (diameter 0) (color 0 0 0 0)
+  )
+  (wire (pts (xy 163.83 58.42) (xy 163.83 62.23))
+    (stroke (width 0) (type default) (color 0 0 0 0))
+  )
+  (wire (pts (xy 163.83 80.01) (xy 163.83 83.82))
+    (stroke (width 0) (type default) (color 0 0 0 0))
+  )
+  (wire (pts (xy 118.11 72.39) (xy 118.11 80.01))
+    (stroke (width 0) (type default) (color 0 0 0 0))
+  )
+  (wire (pts (xy 142.24 58.42) (xy 142.24 62.23))
+    (stroke (width 0) (type default) (color 0 0 0 0))
+  )
+  (wire (pts (xy 163.83 72.39) (xy 163.83 80.01))
+    (stroke (width 0) (type default) (color 0 0 0 0))
+  )
+  (wire (pts (xy 118.11 58.42) (xy 118.11 62.23))
+    (stroke (width 0) (type default) (color 0 0 0 0))
+  )
+  (wire (pts (xy 163.83 80.01) (xy 118.11 80.01))
+    (stroke (width 0) (type default) (color 0 0 0 0))
+  )
+  (wire (pts (xy 142.24 72.39) (xy 142.24 76.2))
+    (stroke (width 0) (type default) (color 0 0 0 0))
+  )
+  (text "Starter button" (at 113.03 54.61 0)
+    (effects (font (size 1.27 1.27)) (justify left bottom))
+  )
+  (text "Launch control" (at 158.75 54.61 0)
+    (effects (font (size 1.27 1.27)) (justify left bottom))
+  )
+  (text "Cockpit EStop" (at 137.16 54.61 0)
+    (effects (font (size 1.27 1.27)) (justify left bottom))
+  )
+  (hierarchical_label "GND" (shape input) (at 163.83 83.82 0)
+    (effects (font (size 1.27 1.27)) (justify left))
+  )
+  (hierarchical_label "Shutdown2" (shape input) (at 142.24 58.42 0)
+    (effects (font (size 1.27 1.27)) (justify left))
+  )
+  (hierarchical_label "Shutdown 1" (shape input) (at 142.24 76.2 0)
+    (effects (font (size 1.27 1.27)) (justify left))
+  )
+  (hierarchical_label "StarterSignal" (shape input) (at 118.11 58.42 0)
+    (effects (font (size 1.27 1.27)) (justify left))
+  )
+  (hierarchical_label "Launch control" (shape input) (at 163.83 58.42 0)
+    (effects (font (size 1.27 1.27)) (justify left))
+  )
+  (symbol (lib_id "Switch:SW_SPST") (at 142.24 67.31 90) (unit 1)
+    (in_bom yes) (on_board yes) (fields_autoplaced)
+    (property "Reference" "SW?" (id 0) (at 143.51 66.0399 90)
+      (effects (font (size 1.27 1.27)) (justify right))
+    )
+    (property "Value" "SW_SPST" (id 1) (at 143.51 68.5799 90)
+      (effects (font (size 1.27 1.27)) (justify right))
+    )
+    (property "Footprint" "" (id 2) (at 142.24 67.31 0)
+      (effects (font (size 1.27 1.27)) hide)
+    )
+    (property "Datasheet" "~" (id 3) (at 142.24 67.31 0)
+      (effects (font (size 1.27 1.27)) hide)
+    )
+    (pin "1")
+    (pin "2")
+  )
+  (symbol (lib_id "Switch:SW_MEC_5G") (at 118.11 67.31 90) (unit 1)
+    (in_bom yes) (on_board yes)
+    (property "Reference" "SW?" (id 0) (at 119.38 66.0399 90)
+      (effects (font (size 1.27 1.27)) (justify right))
+    )
+    (property "Value" "SW_MEC_5G" (id 1) (at 119.38 68.5799 90)
+      (effects (font (size 1.27 1.27)) (justify right))
+    )
+    (property "Footprint" "" (id 2) (at 113.03 67.31 0)
+      (effects (font (size 1.27 1.27)) hide)
+    )
+    (property "Datasheet" "http://www.apem.com/int/index.php?controller=attachment&id_attachment=488" (id 3) (at 113.03 67.31 0)
+      (effects (font (size 1.27 1.27)) hide)
+    )
+    (pin "1")
+    (pin "3")
+    (pin "2")
+    (pin "4")
+  )
+  (symbol (lib_id "Switch:SW_SPST") (at 163.83 67.31 90) (unit 1)
+    (in_bom yes) (on_board yes) (fields_autoplaced)
+    (property "Reference" "SW?" (id 0) (at 165.1 66.0399 90)
+      (effects (font (size 1.27 1.27)) (justify right))
+    )
+    (property "Value" "SW_SPST" (id 1) (at 165.1 68.5799 90)
+      (effects (font (size 1.27 1.27)) (justify right))
+    )
+    (property "Footprint" "" (id 2) (at 163.83 67.31 0)
+      (effects (font (size 1.27 1.27)) hide)
+    )
+    (property "Datasheet" "~" (id 3) (at 163.83 67.31 0)
+      (effects (font (size 1.27 1.27)) hide)
+    )
+    (pin "1")
+    (pin "2")
+  )
 )

Commit message: Added fans and their control circuit. Added some wires.
Parts:
- added SW?: SW_SPST, symbol Switch:SW_SPST
Connections:
- net GND: now also SW?.1 (A)
- new net Fan signal: SW?.2 (B)
Other:
- note added: "Fan override"
- note added: "Serial connector here"
Changed lines of the file:
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@@
+    (stroke (width 0) (type default) (color 0 0 0 0))
+  )
+  (wire (pts (xy 163.83 80.01) (xy 190.5 80.01))
     (stroke (width 0) (type default) (color 0 0 0 0))
   )
   (wire (pts (xy 118.11 72.39) (xy 118.11 80.01))
+    (stroke (width 0) (type default) (color 0 0 0 0))
+  )
+  (wire (pts (xy 190.5 80.01) (xy 190.5 72.39))
+    (stroke (width 0) (type default) (color 0 0 0 0))
+  )
+  (wire (pts (xy 190.5 58.42) (xy 190.5 62.23))
     (stroke (width 0) (type default) (color 0 0 0 0))
   )
@@
     (stroke (width 0) (type default) (color 0 0 0 0))
   )
+  (text "Serial connector here " (at 212.09 53.34 0)
+    (effects (font (size 1.27 1.27)) (justify left bottom))
+  )
   (text "Starter button" (at 113.03 54.61 0)
+    (effects (font (size 1.27 1.27)) (justify left bottom))
+  )
+  (text "Fan override" (at 187.96 54.61 0)
     (effects (font (size 1.27 1.27)) (justify left bottom))
   )
@@
   (text "Cockpit EStop" (at 137.16 54.61 0)
     (effects (font (size 1.27 1.27)) (justify left bottom))
+  )
+  (hierarchical_label "Fan signal" (shape input) (at 190.5 58.42 0)
+    (effects (font (size 1.27 1.27)) (justify left))
   )
   (hierarchical_label "GND" (shape input) (at 163.83 83.82 0)
@@
     (pin "4")
   )
+  (symbol (lib_id "Switch:SW_SPST") (at 190.5 67.31 90) (unit 1)
+    (in_bom yes) (on_board yes) (fields_autoplaced)
+    (property "Reference" "SW?" (id 0) (at 191.77 66.0399 90)
+      (effects (font (size 1.27 1.27)) (justify right))
+    )
+    (property "Value" "SW_SPST" (id 1) (at 191.77 68.5799 90)
+      (effects (font (size 1.27 1.27)) (justify right))
+    )
+    (property "Footprint" "" (id 2) (at 190.5 67.31 0)
+      (effects (font (size 1.27 1.27)) hide)
+    )
+    (property "Datasheet" "~" (id 3) (at 190.5 67.31 0)
+      (effects (font (size 1.27 1.27)) hide)
+    )
+    (pin "1")
+    (pin "2")
+  )
   (symbol (lib_id "Switch:SW_SPST") (at 163.83 67.31 90) (unit 1)

Commit message: Finished wiring up the ECU.
Parts:
- added J?: AudioJack3, symbol Connector:AudioJack3
Connections:
- new net SerialGND: J?.S
- new net SerialRX: J?.R
- new net SerialTX: J?.T
Changed lines of the file:
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@@
   (junction (at 163.83 80.01) (diameter 0) (color 0 0 0 0)
+  )
+  (wire (pts (xy 219.71 68.58) (xy 223.52 68.58))
+    (stroke (width 0) (type default) (color 0 0 0 0))
   )
   (wire (pts (xy 163.83 58.42) (xy 163.83 62.23))
@@
     (stroke (width 0) (type default) (color 0 0 0 0))
   )
+  (wire (pts (xy 219.71 63.5) (xy 223.52 63.5))
+    (stroke (width 0) (type default) (color 0 0 0 0))
+  )
   (wire (pts (xy 163.83 80.01) (xy 190.5 80.01))
     (stroke (width 0) (type default) (color 0 0 0 0))
   )
   (wire (pts (xy 118.11 72.39) (xy 118.11 80.01))
+    (stroke (width 0) (type default) (color 0 0 0 0))
+  )
+  (wire (pts (xy 219.71 66.04) (xy 223.52 66.04))
     (stroke (width 0) (type default) (color 0 0 0 0))
   )
@@
     (effects (font (size 1.27 1.27)) (justify left bottom))
   )
+  (hierarchical_label "SerialRX" (shape input) (at 219.71 66.04 180)
+    (effects (font (size 1.27 1.27)) (justify right))
+  )
   (hierarchical_label "Fan signal" (shape input) (at 190.5 58.42 0)
     (effects (font (size 1.27 1.27)) (justify left))
@@
   (hierarchical_label "Shutdown2" (shape input) (at 142.24 58.42 0)
     (effects (font (size 1.27 1.27)) (justify left))
+  )
+  (hierarchical_label "SerialGND" (shape input) (at 219.71 68.58 180)
+    (effects (font (size 1.27 1.27)) (justify right))
+  )
+  (hierarchical_label "SerialTX" (shape input) (at 219.71 63.5 180)
+    (effects (font (size 1.27 1.27)) (justify right))
   )
   (hierarchical_label "Shutdown 1" (shape input) (at 142.24 76.2 0)
@@
     (pin "2")
   )
+  (symbol (lib_id "Connector:AudioJack3") (at 228.6 66.04 180) (unit 1)
+    (in_bom yes) (on_board yes) (fields_autoplaced)
+    (property "Reference" "J?" (id 0) (at 236.22 64.1349 0)
+      (effects (font (size 1.27 1.27)) (justify right))
+    )
+    (property "Value" "AudioJack3" (id 1) (at 236.22 66.6749 0)
+      (effects (font (size 1.27 1.27)) (justify right))
+    )
+    (property "Footprint" "" (id 2) (at 228.6 66.04 0)
+      (effects (font (size 1.27 1.27)) hide)
+    )
+    (property "Datasheet" "~" (id 3) (at 228.6 66.04 0)
+      (effects (font (size 1.27 1.27)) hide)
+    )
+    (pin "R")
+    (pin "S")
+    (pin "T")
+  )
   (symbol (lib_id "Switch:SW_SPST") (at 163.83 67.31 90) (unit 1)

Commit message: Included BSPD and started adding labels
Connections:
- net SerialRX: now also J?.T; no longer J?.R
- net SerialTX: now also J?.R; no longer J?.T
Other:
- note added: "Serial connector"
- note removed: "Serial connector here"
Changed lines of the file:
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@@
-    (stroke (width 0) (type default) (color 0 0 0 0))
-  )
-  (wire (pts (xy 219.71 63.5) (xy 223.52 63.5))
     (stroke (width 0) (type default) (color 0 0 0 0))
   )
@@
   )
   (wire (pts (xy 118.11 72.39) (xy 118.11 80.01))
+    (stroke (width 0) (type default) (color 0 0 0 0))
+  )
+  (wire (pts (xy 219.71 63.5) (xy 223.52 63.5))
     (stroke (width 0) (type default) (color 0 0 0 0))
   )
@@
     (stroke (width 0) (type default) (color 0 0 0 0))
   )
-  (text "Serial connector here " (at 212.09 53.34 0)
+  (text "Serial connector" (at 218.44 54.61 0)
     (effects (font (size 1.27 1.27)) (justify left bottom))
   )
@@
     (effects (font (size 1.27 1.27)) (justify left bottom))
   )
-  (hierarchical_label "SerialRX" (shape input) (at 219.71 66.04 180)
+  (hierarchical_label "SerialRX" (shape input) (at 219.71 63.5 180)
     (effects (font (size 1.27 1.27)) (justify right))
   )
@@
     (effects (font (size 1.27 1.27)) (justify right))
   )
-  (hierarchical_label "SerialTX" (shape input) (at 219.71 63.5 180)
+  (hierarchical_label "SerialTX" (shape input) (at 219.71 66.04 180)
     (effects (font (size 1.27 1.27)) (justify right))
   )

Commit message: Changed labels to match old wires
Other:
- note added: "Label: Dash Switches Connector type: TBC"
- note added: "Pin1 Pin2 Pin3 Pin4 Pin5 Pin6 Pin7 Pin8"
Changed lines of the file:
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@@
     (stroke (width 0) (type default) (color 0 0 0 0))
+  )
+  (text "Pin1\nPin2\nPin3\nPin4\nPin5\nPin6\nPin7\nPin8\n" (at 47.625 67.31 0)
+    (effects (font (size 1.27 1.27)) (justify left bottom))
   )
   (text "Serial connector" (at 218.44 54.61 0)
@@
     (effects (font (size 1.27 1.27)) (justify left bottom))
   )
+  (text "Label: Dash Switches\nConnector type: TBC" (at 47.625 50.165 0)
+    (effects (font (size 1.27 1.27)) (justify left bottom))
+  )
   (text "Cockpit EStop" (at 137.16 54.61 0)
     (effects (font (size 1.27 1.27)) (justify left bottom))
@@
     (effects (font (size 1.27 1.27)) (justify left))
   )
+  (hierarchical_label "SerialRX" (shape input) (at 53.975 62.23 0)
+    (effects (font (size 1.27 1.27)) (justify left))
+  )
   (hierarchical_label "GND" (shape input) (at 163.83 83.82 0)
+    (effects (font (size 1.27 1.27)) (justify left))
+  )
+  (hierarchical_label "Shutdown2" (shape input) (at 53.975 55.88 0)
+    (effects (font (size 1.27 1.27)) (justify left))
+  )
+  (hierarchical_label "Launch control" (shape input) (at 53.975 57.785 0)
+    (effects (font (size 1.27 1.27)) (justify left))
+  )
+  (hierarchical_label "SerialTX" (shape input) (at 53.975 64.135 0)
     (effects (font (size 1.27 1.27)) (justify left))
   )
@@
     (effects (font (size 1.27 1.27)) (justify right))
   )
+  (hierarchical_label "Fan signal" (shape input) (at 53.975 60.325 0)
+    (effects (font (size 1.27 1.27)) (justify left))
+  )
   (hierarchical_label "SerialTX" (shape input) (at 219.71 66.04 180)
     (effects (font (size 1.27 1.27)) (justify right))
   )
+  (hierarchical_label "SerialGND" (shape input) (at 53.975 66.04 0)
+    (effects (font (size 1.27 1.27)) (justify left))
+  )
   (hierarchical_label "Shutdown 1" (shape input) (at 142.24 76.2 0)
+    (effects (font (size 1.27 1.27)) (justify left))
+  )
+  (hierarchical_label "StarterSignal" (shape input) (at 53.975 52.07 0)
     (effects (font (size 1.27 1.27)) (justify left))
   )
@@
     (effects (font (size 1.27 1.27)) (justify left))
   )
+  (hierarchical_label "Shutdown 1" (shape input) (at 53.975 53.975 0)
+    (effects (font (size 1.27 1.27)) (justify left))
+  )

Commit message: Added connector pinouts
Connections:
- net GND: no longer SW?.1 (A), SW?.2 (A)
- net StarterSignal renamed Fused 12V
- new net StartSignal: SW?.1 (A), SW?.2 (A)
Other:
- note added: "Label: Dash Switches Connector type: Deutsch 12 pin Connector label: Dash switches"
- note added: "Pin1 Pin2 Pin3 Pin4 Pin5 Pin6 Pin7 Pin8 Pin9"
- note removed: "Label: Dash Switches Connector type: TBC"
- note removed: "Pin1 Pin2 Pin3 Pin4 Pin5 Pin6 Pin7 Pin8"
Changed lines of the file:
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@@
-    (stroke (width 0) (type default) (color 0 0 0 0))
-  )
-  (wire (pts (xy 118.11 72.39) (xy 118.11 80.01))
     (stroke (width 0) (type default) (color 0 0 0 0))
   )
@@
     (stroke (width 0) (type default) (color 0 0 0 0))
   )
-  (wire (pts (xy 163.83 80.01) (xy 118.11 80.01))
-    (stroke (width 0) (type default) (color 0 0 0 0))
-  )
   (wire (pts (xy 142.24 72.39) (xy 142.24 76.2))
     (stroke (width 0) (type default) (color 0 0 0 0))
   )
-  (text "Pin1\nPin2\nPin3\nPin4\nPin5\nPin6\nPin7\nPin8\n" (at 47.625 67.31 0)
+  (text "Pin1\nPin2\nPin3\nPin4\nPin5\nPin6\nPin7\nPin8\nPin9" (at 47.625 67.31 0)
     (effects (font (size 1.27 1.27)) (justify left bottom))
   )
@@
     (effects (font (size 1.27 1.27)) (justify left bottom))
   )
-  (text "Label: Dash Switches\nConnector type: TBC" (at 47.625 50.165 0)
+  (text "Label: Dash Switches\nConnector type: Deutsch 12 pin\nConnector label: Dash switches\n"
+    (at 47.498 47.752 0)
     (effects (font (size 1.27 1.27)) (justify left bottom))
   )
@@
     (effects (font (size 1.27 1.27)) (justify left))
   )
-  (hierarchical_label "SerialRX" (shape input) (at 53.975 62.23 0)
+  (hierarchical_label "Fused 12V" (shape input) (at 118.11 58.42 0)
+    (effects (font (size 1.27 1.27)) (justify left))
+  )
+  (hierarchical_label "SerialRX" (shape input) (at 53.34 62.484 0)
+    (effects (font (size 1.27 1.27)) (justify left))
+  )
+  (hierarchical_label "Fused 12V" (shape input) (at 53.086 49.784 0)
     (effects (font (size 1.27 1.27)) (justify left))
   )
@@
     (effects (font (size 1.27 1.27)) (justify left))
   )
-  (hierarchical_label "Shutdown2" (shape input) (at 53.975 55.88 0)
+  (hierarchical_label "Shutdown2" (shape input) (at 53.34 56.134 0)
     (effects (font (size 1.27 1.27)) (justify left))
   )
-  (hierarchical_label "Launch control" (shape input) (at 53.975 57.785 0)
+  (hierarchical_label "Launch control" (shape input) (at 53.34 58.039 0)
     (effects (font (size 1.27 1.27)) (justify left))
   )
-  (hierarchical_label "SerialTX" (shape input) (at 53.975 64.135 0)
+  (hierarchical_label "SerialTX" (shape input) (at 53.34 64.389 0)
     (effects (font (size 1.27 1.27)) (justify left))
   )
@@
     (effects (font (size 1.27 1.27)) (justify right))
   )
-  (hierarchical_label "Fan signal" (shape input) (at 53.975 60.325 0)
+  (hierarchical_label "Fan signal" (shape input) (at 53.34 60.579 0)
     (effects (font (size 1.27 1.27)) (justify left))
   )
@@
     (effects (font (size 1.27 1.27)) (justify right))
   )
-  (hierarchical_label "SerialGND" (shape input) (at 53.975 66.04 0)
+  (hierarchical_label "SerialGND" (shape input) (at 53.34 66.294 0)
     (effects (font (size 1.27 1.27)) (justify left))
   )
@@
     (effects (font (size 1.27 1.27)) (justify left))
   )
-  (hierarchical_label "StarterSignal" (shape input) (at 53.975 52.07 0)
+  (hierarchical_label "StartSignal" (shape input) (at 53.34 52.324 0)
     (effects (font (size 1.27 1.27)) (justify left))
   )
-  (hierarchical_label "StarterSignal" (shape input) (at 118.11 58.42 0)
+  (hierarchical_label "StartSignal" (shape input) (at 118.11 72.39 0)
     (effects (font (size 1.27 1.27)) (justify left))
   )
@@
     (effects (font (size 1.27 1.27)) (justify left))
   )
-  (hierarchical_label "Shutdown 1" (shape input) (at 53.975 53.975 0)
+  (hierarchical_label "Shutdown 1" (shape input) (at 53.34 54.229 0)
     (effects (font (size 1.27 1.27)) (justify left))
   )
