File: Loom23/Loom.kicad_sch (KiCad schematic)
At the start: 8 parts

Commit message: Added connector pinouts
Other:
- removed sheet Oil pressure sensor
- removed sheet Ride height sensors (4x)
- removed sheet Telemetry
- removed sheet Wheel speed sensors (4x)
